File: examples/infrared-transceiver/infrared-transceiver.kicad_sch (KiCad schematic)
At the start: 11 parts, among them Q1 S8050, U1 TXMCU

Commit message: fix: support hierarchical KiCad net names
Parts:
- 1111: renamed from ?; footprint infrared-transceiver-easyedapro: -> (none)
- C1: footprint infrared-transceiver-easyedapro:C0603 -> Capacitor_THT:C_Disc_D3.0mm_W1.6mm_P2.50mm
- H1: footprint infrared-transceiver-easyedapro:HDR-TH_4P-P2.54-V-M -> Connector:FanPinHeader_1x04_P2.54mm_Vertical
- IR1: footprint infrared-transceiver-easyedapro:LED-TH_BD5.9-P2.54-RD_WHITE -> LED_THT:LED_D5.0mm
- LED1: footprint infrared-transceiver-easyedapro:SENSOR-TG_TSOP38236 -> LED_THT:LED_D5.0mm-3
- LED2: footprint infrared-transceiver-easyedapro:LED0603-FD -> LED_THT:LED_D5.0mm
- Q1: footprint infrared-transceiver-easyedapro:SOT-23-3_L2.9-W1.3-P1.90-LS2.3-BR -> Package_TO_SOT_THT:TO-92L_Inline_Wide
- R1, R2, R3: footprint infrared-transceiver-easyedapro:R0603 -> Resistor_THT:R_Axial_DIN0207_L6.3mm_D2.5mm_P10.16mm_Horizontal
- U1: footprint infrared-transceiver-easyedapro: -> Package_DIP:CERDIP-8_W7.62mm_SideBrazed
Connections:
- net GND: now also U1.8 (GND)
- net RX: now also U1.5 (IO5)
- net TX: now also U1.4 (IO4)
- net VCC: now also U1.1 (VIN)
- net at R3.1: now also U1.7 (IO7)
- net at U1.3 (IO3): now also LED2.2 (C)
- net at U1.6 (IO6): now also LED1.1 (OUT)
Other:
- moved on the sheet: C1, IR1, LED1, LED2, Q1, R1, R2, R3, U1
