File: examples/tm1637-display-module/tm1637-display-module.kicad_pcb (KiCad board)
At the start: 2 copper layers, 8 parts

Commit message: chore(examples): refresh test fixtures
Parts:
- H1, U4: footprint Connector:FanPinHeader_1x04_P2.54mm_Vertical -> Connector_PinHeader_2.54mm:PinHeader_1x04_P2.54mm_Vertical
- moved C4 42.8 mm to (167.5, 125.8)
- moved C3 42.8 mm to (167.5, 122.6)
- moved H1 17.8 mm to (159.0, 123.3)
- moved U4 17.4 mm to (163.6, 123.3)
- moved R4 15.4 mm to (158.3, 115.0)
- moved R5 15.4 mm to (158.3, 119.0)
- moved LED1 13.6 mm to (138.8, 105.6)
- moved U3 13.6 mm to (158.3, 88.0)
